File: esp32-prog.kicad_pcb (KiCad board)
At the start: 4 copper layers, 43 x 21.8 mm, 17 parts, among them J1 USB_C_Receptacle_USB2.0, J2 ESP_PROG, J3 POWER, J4 DTR_RTS, Q1 S8050, Q2 S8050, U1 CH340B, U2 AP1117-33

Commit message: Finalise Rev 1.2
Parts:
- renumbered REF** to LOGO
